File: goldberg/generated_pcb/middle/middle.kicad_pcb (KiCad board)
At the start: 2 copper layers, 116 x 115.3 mm, 44 parts, among them SW1 switch, SW10 switch, SW11 switch, SW12 switch, SW13 switch, SW14 switch, SW15-1 switch, SW15-2 switch, SW16 switch, SW17 switch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

Commit message: PC change
Parts:
- removed the G*** at (76.2, 48.3)
- added JP1: L_GND, footprints:Jumper, F.Cu at (129.5, 55.4)
- added JP2: L_VCC, footprints:Jumper, F.Cu at (127.0, 55.4)
- added JP3: L_SCL, footprints:Jumper, F.Cu at (124.5, 55.4)
- added JP4: L_SDA, footprints:Jumper, F.Cu at (121.9, 55.4)
- added JP5: R_GND, footprints:Jumper, B.Cu at (129.5, 55.4)
- added JP6: R_VCC, footprints:Jumper, B.Cu at (127.0, 55.4)
- added JP7: R_SCL, footprints:Jumper, B.Cu at (124.5, 55.4)
- added JP8: R_SDA, footprints:Jumper, B.Cu at (121.9, 55.4)
- added LED1: WS2812B, footprints:LED_WS2812B_4Pad, F.Cu at (108.6, 36.8)
- added LED10: WS2812B, footprints:LED_WS2812B_4Pad, F.Cu at (104.8, 78.1)
- added LED2: WS2812B, footprints:LED_WS2812B_4Pad, F.Cu at (89.5, 36.2)
- added LED3: WS2812B, footprints:LED_WS2812B_4Pad, F.Cu at (66.7, 29.2)
- added LED4: WS2812B, footprints:LED_WS2812B_4Pad, F.Cu at (47.0, 35.6)
- added LED5: WS2812B, footprints:LED_WS2812B_4Pad, F.Cu at (33.0, 47.0)
- added LED6: WS2812B, footprints:LED_WS2812B_4Pad, F.Cu at (33.0, 66.7)
- added LED7: WS2812B, footprints:LED_WS2812B_4Pad, F.Cu at (52.1, 76.2)
- added LED8: WS2812B, footprints:LED_WS2812B_4Pad, F.Cu at (73.0, 85.1)
- added LED9: WS2812B, footprints:LED_WS2812B_4Pad, F.Cu at (85.1, 78.1)
- added P1: OLED, footprints:SSD_1306_128x32, B.Cu at (129.5, 58.4)
- added R1: 4.7K, Resistor_THT:R_Axial_DIN0207_L6.3mm_D2.5mm_P10.16mm_Horizontal, F.Cu at (121.9, 77.5)
- added R2: 4.7K, Resistor_THT:R_Axial_DIN0207_L6.3mm_D2.5mm_P10.16mm_Horizontal, F.Cu at (121.9, 82.5)
- added SW15: SW_Push, Button_Switch_THT:SW_PUSH_6mm_H5mm, B.Cu at (33.1, 25.4)
- added SW19: SW_Push, Button_Switch_THT:SW_PUSH_6mm_H5mm, F.Cu at (26.7, 25.4)
- U2: value ProMicro -> promicro-squiggle
- moved U2 0.19 mm to (125.7, 39.4)
Connections:
- U1 pad 1: SDA -> VCC
- U1 pad 2: Net-(U1-Pad2) -> GND
- U1 pad 3: Net-(U1-Pad3) -> DATA
- U1 pad 4: (no net) -> Net-(U1-Pad4)
- U2 pad 1: (no net) -> LED
- U2 pad 17: (no net) -> Net-(U2-Pad17)
- U2 pad 18: (no net) -> Net-(U2-Pad18)
- U2 pad 19: (no net) -> Net-(U2-Pad19)
- U2 pad 2: (no net) -> DATA
- U2 pad 20: (no net) -> Net-(U2-Pad20)
- U2 pad 21: Net-(U1-Pad2) -> VCC
- U2 pad 22: (no net) -> Net-(SW15-Pad2)
- U2 pad 23: Net-(U1-Pad3) -> GND
- U2 pad 24: (no net) -> Net-(U2-Pad24)
- U2 pad 3: (no net) -> GND
- U2 pad 4: (no net) -> GND
- U2 pad 5: (no net) -> SDA
- U2 pad 6: SDA -> SCL
- U2 pad 7: (no net) -> Net-(U2-Pad7)
Routing:
- net GND: track 0.00 -> 412.4 mm, vias 0 -> 19
- net VCC: track 0.00 -> 378.1 mm, vias 0 -> 19
- net Net-(SW15-Pad2): track 0.00 -> 104.6 mm
- net Net-(U1-Pad2): track 58.9 -> 0.00 mm
- net SCL: track 0.00 -> 54.0 mm, vias 0 -> 2
- net Net-(U1-Pad3): track 53.6 -> 0.00 mm
- net Net-(LED7-Pad2): track 0.00 -> 45.3 mm, vias 0 -> 2
- net DATA: track 0.00 -> 42.1 mm, vias 0 -> 2
- net Net-(LED6-Pad2): track 0.00 -> 37.4 mm, vias 0 -> 4
- net Net-(LED2-Pad2): track 0.00 -> 37.2 mm, vias 0 -> 4
- net Net-(LED10-Pad4): track 0.00 -> 33.8 mm, vias 0 -> 2
- net LED: track 0.00 -> 31.1 mm, vias 0 -> 2
- net Net-(JP3-Pad1): track 0.00 -> 29.6 mm, vias 0 -> 3
- net Net-(LED1-Pad2): track 0.00 -> 27.1 mm, vias 0 -> 2
- net LED_CONT: track 0.00 -> 26.8 mm, vias 0 -> 4
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